File: kicad/diff-probe.kicad_pcb (KiCad board)
At the start: 2 copper layers, 50 x 12 mm, 29 parts, among them IC3 LMH6702, IC4 LMH6702, IC5 LMH6702, J3 HEADER-1X2CARD-EDGE, J4 CON-1X3-TAB-AMP-29173-3-NARROW, X2 SMA--BU-SMA-H

Commit message: Updates
Parts:
- C13, C14, C15, C16, C17, C18, C19, C20, C21, C22, C23, C24: footprint diff-probe:0402-SQUARE -> Capacitor_SMD:C_0402_1005Metric
- C52, C54: footprint diff-probe:0603 -> Capacitor_SMD:C_0603_1608Metric
- IC3, IC4, IC5: footprint diff-probe:SO08 -> Package_SO:SOIC-8_3.9x4.9mm_P1.27mm
- R20, R22, R26, R27, R28, R30, R32, R37, R38: footprint diff-probe:0402-SQUARE -> Resistor_SMD:R_0402_1005Metric
- turned IC3 to 0 degrees
- turned IC4 to 0 degrees
- turned IC5 to 0 degrees
Routing:
- net V+: track 82.2 -> 82.8 mm, vias 3 -> 4
- net GND: track 15.5 -> 14.9 mm, vias 19 -> 18
