File: kicad/diff-probe.kicad_sch (KiCad schematic)
At the start: 29 parts, among them IC3 LMH6702, IC4 LMH6702, IC5 LMH6702, J3 HEADER-1X2CARD-EDGE, J4 CON-1X3-TAB-AMP-29173-3-NARROW, X2 SMA--BU-SMA-H

Commit message: Updates
Parts:
- C13, C14, C15, C16, C17, C18, C19, C20, C21, C22, C23, C24: footprint 0402-SQUARE -> Capacitor_SMD:C_0402_1005Metric
- C52, C54: footprint 0603 -> Capacitor_SMD:C_0603_1608Metric
- IC3, IC4, IC5: footprint SO08 -> Package_SO:SOIC-8_3.9x4.9mm_P1.27mm
- R20, R22, R26, R27, R28, R30, R32, R37, R38: footprint 0402-SQUARE -> Resistor_SMD:R_0402_1005Metric
